Commit message: Add realsense_gazebo_plugin as part of main robotis_ws repo

File: src/open_manipulator/open_manipulator_description/urdf/open_manipulator.gazebo.xacro (robot description, xacro)
@@ -50,41 +50,25 @@
     </plugin>
   </gazebo>
-  <!-- camera -->
-  <gazebo reference="camera_link">
-    <sensor type="camera" name="intel_realsense_r200">
-      <update_rate>30.0</update_rate>
-      <camera name="head">
-        <horizontal_fov>1.02974</horizontal_fov>
+  <!-- RealSense D435 Gazebo Plugin -->
+  <!-- Gazebo Plugin (matches RealSense defaults) -->
+  <gazebo reference="fixed_camera_link">
+    <sensor type="camera" name="d435_camera">
+      <update_rate>30</update_rate>
+      <camera>
+        <horizontal_fov>1.0472</horizontal_fov> <!-- 60° -->
         <image>
-          <width>1920</width>
-          <height>1080</height>
-          <format>R8G8B8</format>
+          <width>640</width>
+          <height>480</height>
         </image>
         <clip>
-          <near>0.02</near>
-          <far>300</far>
+          <near>0.01</near>  <!-- 2cm min range -->
+          <far>1.0</far>     <!-- 2m max range -->
         </clip>
-        <noise>
-          <type>gaussian</type>
-          <!-- Noise is sampled independently per pixel on each frame.
-               That pixel's noise value is added to each of its color
-               channels, which at that point lie in the range [0,1]. -->
-          <mean>0.0</mean>
-          <stddev>0.007</stddev>
-        </noise>
       </camera>
-      <plugin name="camera_controller" filename="libgazebo_ros_camera.so">
+      <plugin name="camera_plugin" filename="libgazebo_ros_camera.so">
         <alwaysOn>true</alwaysOn>
-        <updateRate>0.0</updateRate>
-        <cameraName>camera/color</cameraName>
-        <imageTopicName>image_raw</imageTopicName>
-        <cameraInfoTopicName>camera_info</cameraInfoTopicName>
-        <frameName>camera_link</frameName>
-        <hackBaseline>0.07</hackBaseline>
-        <distortionK1>0.0</distortionK1>
-        <distortionK2>0.0</distortionK2>
-        <distortionK3>0.0</distortionK3>
-        <distortionT1>0.0</distortionT1>
-        <distortionT2>0.0</distortionT2>
+        <cameraName>d435</cameraName>
+        <imageTopicName>color/image_raw</imageTopicName>
+        <frameName>fixed_camera_link</frameName>
       </plugin>
     </sensor>

File: src/open_manipulator/open_manipulator_description/urdf/open_manipulator.urdf.xacro (robot description, xacro)
@@ -1,4 +1,3 @@
-<?xml version="1.0"?>
-<!-- Open_Manipulator Chain -->
+<?xml version="1.0"?> <!-- Open_Manipulator Chain -->
 <robot xmlns:xacro="http://ros.org/wiki/xacro">
   <!-- Link 1 -->
@@ -235,4 +234,24 @@
     </inertial>
   </link>
+  <xacro:include filename="$(find realsense2_description)/urdf/_d435.urdf.xacro"/>
+  <link name="fixed_camera_link">
+    <visual>
+      <origin xyz="0 0 0" rpy="0 0 0"/>
+      <geometry>
+        <box size="0.01 0.01 0.01"/>
+      </geometry>
+      <material name="red"/>
+    </visual>
+  </link>
+  <!-- Fixed Camera Joint -->
+  <joint name="fixed_camera_joint" type="fixed">
+    <origin xyz="0.07 0.012 0.032" rpy="0 0 0"/>
+    <parent link="link5"/>
+    <child link="fixed_camera_link"/>
+  </joint>
+  <!-- RealSense D435 Sensor -->
+  <xacro:sensor_d435 parent="fixed_camera_link" name="d435" use_nominal_extrinsics="true">
+    <origin xyz="0 0 0" rpy="0 0 0"/>
+  </xacro:sensor_d435>
   <!-- Realsense Camera Joint Position -->
 <!--   <joint name="camera_joint" type="fixed">
